Commit message: feat: improved RL model with wider workspace and two-phase training
- Shoulder pitch ROM ±45° → ±60° for better reachability
- Workspace: max radius 0.525m, Z range 0.10-0.585m
- 35% edge-biased target sampling, 85% start randomization
- Two-phase training: 1M budget + phase 2 hunts for 99%+ rolling SR
- Direct SR tracking from episode outcomes (bypasses SB3 logger timing)
- Server: matched threshold to training (0.05m), starts from last position
- Frontend: proper cylindrical workspace clamping with hollow core,
  thick trail line (Line2), larger spheres, updated title
- Fixed training curve graph to use latest tfevents only
- Added scripts/eval_spatial.py for spatial evaluation

Co-Authored-By: Claude Opus 4.6 (1M context) <noreply@anthropic.com>

File: robot_arm/robot_arm.urdf (robot description, URDF)
Before this commit: robot three_link_arm, 5 links, 4 joints
Joints:
- joint joint_1: limit lower=-0.785 upper=0.785 effort=100 velocity=2.0 -> lower=-1.047 upper=1.047 effort=100 velocity=2.0
